File: Pavel/Powere.sch (KiCad schematic (older format))
At the start: 15 parts, among them U201 TPS63031

Commit message: save work at oth
Parts:
- FB201, FB202, FB203: symbol Pavel_privat:742792641 -> Tuerschild_Boarddesign-rescue:742792641-Pavel_privat
- U201: symbol Pavel_privat:TPS63031 -> Tuerschild_Boarddesign-rescue:TPS63031-Pavel_privat
Changed lines of the file:
@@
 EESchema Schematic File Version 4
 LIBS:Tuerschild_Boarddesign-cache
-EELAYER 30 0
+EELAYER 29 0
 EELAYER END
 $Descr A4 11693 8268
@@
 $EndDescr
 $Comp
-L Pavel_privat:TPS63031 U?
+L Tuerschild_Boarddesign-rescue:TPS63031-Pavel_privat U?
 U 1 1 5DC4BD48
 P 5700 4700
@@
 	6200 4500 6350 4500
 $Comp
-L Pavel_privat:742792641 FB202
+L Tuerschild_Boarddesign-rescue:742792641-Pavel_privat FB202
 U 1 1 5DD8ABAB
 P 5700 2100
+AR Path="/5DD8ABAB" Ref="FB202"  Part="1"
+AR Path="/5DC46C2E/5DD8ABAB" Ref="FB202"  Part="1"
 F 0 "FB202" H 5700 2250 60  0000 C CNN
 F 1 "742792641" H 5700 2350 60  0001 C CNN
@@
 	5900 2100 6250 2100
 $Comp
-L Pavel_privat:742792641 FB203
+L Tuerschild_Boarddesign-rescue:742792641-Pavel_privat FB203
 U 1 1 5DD8E51F
 P 5700 2400
+AR Path="/5DD8E51F" Ref="FB203"  Part="1"
+AR Path="/5DC46C2E/5DD8E51F" Ref="FB203"  Part="1"
 F 0 "FB203" H 5700 2250 60  0000 C CNN
 F 1 "742792641" H 5700 2250 60  0001 C CNN
@@
 $EndComp
 $Comp
-L Pavel_privat:742792641 FB201
+L Tuerschild_Boarddesign-rescue:742792641-Pavel_privat FB201
 U 1 1 5DD92A84
 P 3600 4500
+AR Path="/5DD92A84" Ref="FB201"  Part="1"
+AR Path="/5DC46C2E/5DD92A84" Ref="FB201"  Part="1"
 F 0 "FB201" H 3600 4350 60  0000 C CNN
 F 1 "742792641" H 3600 4350 60  0001 C CNN

Commit message: save commit again
Parts:
- added R502, R504: 0, Resistor_SMD:R_0603_1608Metric_Pad1.05x0.95mm_HandSolder, symbol Device:R
- added R503: 100k, Resistor_SMD:R_0603_1608Metric_Pad1.05x0.95mm_HandSolder, symbol Device:R
- added TP501, TP502, TP503, TP504, TP505, TP506: Testpunkt_small, TestPoint:TestPoint_Pad_D1.5mm, symbol Pavel_privat:Testpunkt_small
- FB501: renamed from FB201; symbol Tuerschild_Boarddesign-rescue:742792641-Pavel_privat -> Pavel_privat:742792641
- FB502: renamed from FB202; symbol Tuerschild_Boarddesign-rescue:742792641-Pavel_privat -> Pavel_privat:742792641
- FB503: renamed from FB203; symbol Tuerschild_Boarddesign-rescue:742792641-Pavel_privat -> Pavel_privat:742792641
- U501: renamed from U201; symbol Tuerschild_Boarddesign-rescue:TPS63031-Pavel_privat -> Pavel_privat:TPS63031
- renumbered C201 to C501, C202 to C502, C203 to C503, C204 to C504, C205 to C505, C207 to C506, C206 to C507, C208 to C508, C209 to C509, L201 to L501, R201 to R501
Connections:
- net +3.3V: now also R502.1, R504.1, R504.2, TP505.1; no longer U501.10 (FB)
- net +BATT: now also TP501.1
- net +VIN_F: now also TP503.1
- net GND: now also R503.2, TP504.1, TP506.1
- net GNDPWR: now also TP502.1
- new net: R502.2, R503.1, U501.10 (FB)
Other:
- note added: "Messwiderstand für Strommessungen\n"
- note added: "R202,203 für TPS63030"
- moved on the sheet: C507, C508, C509
