File: Pavel/Tuerschild_Boarddesign.kicad_pcb (KiCad board)
At the start: 2 copper layers, 6 parts, among them U101 ESP32-WROOM-32U, U102 TPS63031

Commit message: save commit again
Parts:
- removed C101, C103, C104: 10uF, Capacitor_SMD:C_0603_1608Metric
- removed C102: 0,1uF, Capacitor_SMD:C_0603_1608Metric
- removed U101: ESP32-WROOM-32U, RF_Module:ESP32-WROOM-32U
- removed U102: TPS63031, Pavel_privat:Texas_TPS6303x_ThermalVias
- added C201: 10uF, Capacitor_SMD:C_0603_1608Metric, F.Cu at (151.8, 66.1)
- added C202: 0,1uF, Capacitor_SMD:C_0603_1608Metric, F.Cu at (143.4, 74.7)
- added C203: 0,1uF, Capacitor_SMD:C_0603_1608Metric, F.Cu at (156.2, 63.5)
- added C204: C, Capacitor_SMD:C_0603_1608Metric, F.Cu at (148.9, 71.5)
- added C205: 1uF, Capacitor_SMD:C_0603_1608Metric, F.Cu at (153.2, 68.6)
- added C206: 0,1uF, Capacitor_SMD:C_0603_1608Metric, F.Cu at (156.2, 66.0)
- added C301: 4.7uF, Capacitor_SMD:C_0603_1608Metric, F.Cu at (191.9, 56.1)
- added C302: 4.7uF, Capacitor_SMD:C_0603_1608Metric, F.Cu at (184.2, 64.2)
- added C303: 1uF, Capacitor_SMD:C_0603_1608Metric, F.Cu at (182.2, 66.7)
- added C304: 1uF, Capacitor_SMD:C_0603_1608Metric, F.Cu at (188.5, 60.7)
- added C305: 1uF, Capacitor_SMD:C_0603_1608Metric, F.Cu at (188.5, 63.2)
- added C306: 0.1uF, Capacitor_SMD:C_0603_1608Metric, F.Cu at (186.2, 66.7)
- added C307: 1uF, Capacitor_SMD:C_0603_1608Metric, F.Cu at (192.5, 61.1)
- added C308: 1uF, Capacitor_SMD:C_0603_1608Metric, F.Cu at (190.2, 65.7)
- added C309: 1uF, Capacitor_SMD:C_0603_1608Metric, F.Cu at (194.2, 63.6)
- added C310: 1uF, Capacitor_SMD:C_0603_1608Metric, F.Cu at (194.2, 66.1)
- added C311: 1uF, Capacitor_SMD:C_0603_1608Metric, F.Cu at (192.5, 58.6)
- added C312: 1uF, Capacitor_SMD:C_0603_1608Metric, F.Cu at (178.2, 66.7)
- added C401: Spare, Capacitor_SMD:C_0603_1608Metric, F.Cu at (198.8, 75.8)
- added C402: Spare, Capacitor_SMD:C_0603_1608Metric, F.Cu at (198.8, 78.3)
- added C501: 10uF, Capacitor_SMD:C_0603_1608Metric, F.Cu at (138.8, 96.6)
- added C502: 0,1uF, Capacitor_SMD:C_0603_1608Metric, F.Cu at (140.4, 96.6)
- added C503: 10uF, Capacitor_SMD:C_0805_2012Metric_Pad1.15x1.40mm_HandSolder, F.Cu at (124.9, 96.4)
- added C504: 100nF, Capacitor_SMD:C_0603_1608Metric, F.Cu at (126.7, 96.4)
- added C505: 10uF, Capacitor_SMD:C_0805_2012Metric_Pad1.15x1.40mm_HandSolder, F.Cu at (132.7, 96.3)
- added C506: 100nF, Capacitor_SMD:C_0603_1608Metric, F.Cu at (130.9, 96.4)
- added C507: 10uF, Capacitor_SMD:C_0603_1608Metric, F.Cu at (164.5, 89.5)
- added C508: 10uF, Capacitor_SMD:C_0603_1608Metric, F.Cu at (168.5, 85.8)
- added C509: 0,1uF, Capacitor_SMD:C_0603_1608Metric, F.Cu at (173.6, 82.8)
- added D301: MBR0530, Diode_SMD:D_SOD-123, F.Cu at (169.2, 62.1)
- added D302: MBR0530, Diode_SMD:D_SOD-123, F.Cu at (188.3, 53.2)
- added D303: MBR0530, Diode_SMD:D_SOD-123, F.Cu at (174.9, 62.1)
- added FB201: 742792641, digikey-footprints:0603, F.Cu at (161.3, 52.7)
- added FB501: 742792641, digikey-footprints:0603, F.Cu at (135.0, 97.4)
- added FB502: 742792641, digikey-footprints:0603, F.Cu at (128.8, 97.2)
- added FB503: 742792641, digikey-footprints:0603, F.Cu at (128.8, 95.6)
- added J101: Conn_01x02_Male, Pavel_privat:Batterieeinspeisungspads, F.Cu at (110.8, 97.4)
- added J201: Conn_01x03_Male, Connector:FanPinHeader_1x03_P2.54mm_Vertical, F.Cu at (142.4, 63.4)
- added J301: FH12-24S-0.5SH_E-Ink-Display, Pavel_privat:Hirose_FH12-24S-0.5SH_1x24-1MP_P0.50mm_Horizontal, F.Cu at (175.9, 55.0)
- added L301: 10uH, Pavel_privat:NLCV32-EF, F.Cu at (169.0, 65.6)
- added L501: 1,5uH, Pavel_privat:LPS3015_Coilcraft, F.Cu at (158.5, 83.3)
- added Q301: BC817-25LT1G, Package_TO_SOT_SMD:SOT-23, F.Cu at (187.7, 57.1)
- added Q302: SI1308EDL-T1GE3, Package_TO_SOT_SMD:SOT-323_SC-70, F.Cu at (173.9, 65.6)
- added Q401: BC847BW_135, Package_TO_SOT_SMD:SOT-323_SC-70_Handsoldering, F.Cu at (191.0, 73.8)
- added R201: 10k, Resistor_SMD:R_0603_1608Metric_Pad1.05x0.95mm_HandSolder, F.Cu at (159.3, 58.5)
- added R202: 10k, Resistor_SMD:R_0603_1608Metric_Pad1.05x0.95mm_HandSolder, F.Cu at (149.0, 69.0)
- added R203: R, Resistor_SMD:R_0603_1608Metric_Pad1.05x0.95mm_HandSolder, F.Cu at (152.0, 63.6)
- added R204: R, Resistor_SMD:R_0603_1608Metric_Pad1.05x0.95mm_HandSolder, F.Cu at (156.3, 61.0)
- added R205: R, Resistor_SMD:R_0603_1608Metric_Pad1.05x0.95mm_HandSolder, F.Cu at (155.0, 58.5)
- added R206: R, Resistor_SMD:R_0603_1608Metric_Pad1.05x0.95mm_HandSolder, F.Cu at (126.1, 74.2)
- added R207: R, Resistor_SMD:R_0603_1608Metric_Pad1.05x0.95mm_HandSolder, F.Cu at (152.0, 61.1)
- added R208: 10k, Resistor_SMD:R_0603_1608Metric_Pad1.05x0.95mm_HandSolder, F.Cu at (130.5, 74.2)
- added R209: 0, Resistor_SMD:R_0603_1608Metric_Pad1.05x0.95mm_HandSolder, F.Cu at (134.8, 74.2)
- added R210: 10k, Resistor_SMD:R_0603_1608Metric_Pad1.05x0.95mm_HandSolder, F.Cu at (139.2, 74.7)
- added R211: R, Resistor_SMD:R_0603_1608Metric_Pad1.05x0.95mm_HandSolder, F.Cu at (121.8, 74.2)
- added R301: 4.7k, Resistor_SMD:R_0603_1608Metric_Pad1.05x0.95mm_HandSolder, F.Cu at (180.0, 64.2)
- added R302: 47k, Resistor_SMD:R_0603_1608Metric_Pad1.05x0.95mm_HandSolder, F.Cu at (184.3, 61.7)
- added R303: 10k, Resistor_SMD:R_0603_1608Metric_Pad1.05x0.95mm_HandSolder, F.Cu at (193.4, 52.8)
- added R304: 0.47, Resistor_SMD:R_0603_1608Metric_Pad1.05x0.95mm_HandSolder, F.Cu at (180.0, 61.7)
- added R401: 4.7k, Resistor_SMD:R_0603_1608Metric_Pad1.05x0.95mm_HandSolder, F.Cu at (190.3, 76.9)
- added R402: 47k, Resistor_SMD:R_0603_1608Metric_Pad1.05x0.95mm_HandSolder, F.Cu at (200.5, 73.3)
- added R403: 1.5M, Resistor_SMD:R_0603_1608Metric_Pad1.05x0.95mm_HandSolder, F.Cu at (194.6, 76.9)
- added R404: 1M, Resistor_SMD:R_0603_1608Metric_Pad1.05x0.95mm_HandSolder, F.Cu at (196.1, 73.3)
- added R501: 10k, Resistor_SMD:R_0603_1608Metric_Pad1.05x0.95mm_HandSolder, F.Cu at (169.5, 82.8)
- added R502: 0, Resistor_SMD:R_0603_1608Metric_Pad1.05x0.95mm_HandSolder, F.Cu at (159.9, 92.4)
- added R503: 100k, Resistor_SMD:R_0603_1608Metric_Pad1.05x0.95mm_HandSolder, F.Cu at (164.7, 83.3)
- added R504: 0, Resistor_SMD:R_0603_1608Metric_Pad1.05x0.95mm_HandSolder, F.Cu at (169.5, 80.3)
- added SW201: 219-2MS, Button_Switch_SMD:SW_DIP_SPSTx02_Slide_6.7x6.64mm_W8.61mm_P2.54mm_LowProfile, F.Cu at (146.5, 55.7)
- added SW202: 1977066-1, Pavel_privat:TE_1977066-1, F.Cu at (156.2, 54.4)
- added SW203: 1977066-1, Pavel_privat:TE_1977066-1, F.Cu at (143.5, 70.7)
- added TP501: Testpunkt_small, TestPoint:TestPoint_Pad_D1.5mm, F.Cu at (182.9, 89.9)
- added TP502: Testpunkt_small, TestPoint:TestPoint_Pad_D1.5mm, F.Cu at (182.5, 93.5)
- added TP503: Testpunkt_small, TestPoint:TestPoint_Pad_D1.5mm, F.Cu at (177.4, 80.9)
- added TP504: Testpunkt_small, TestPoint:TestPoint_Pad_D1.5mm, F.Cu at (177.4, 84.4)
- added TP505: Testpunkt_small, TestPoint:TestPoint_Pad_D1.5mm, F.Cu at (176.6, 92.0)
- added TP506: Testpunkt_small, TestPoint:TestPoint_Pad_D1.5mm, F.Cu at (185.9, 90.1)
- added U201: ESP32-WROOM-32U, RF_Module:ESP32-WROOM-32U, F.Cu at (129.9, 61.9)
- added U501: TPS63031, Pavel_privat:Texas_TPS6303x_ThermalVias, F.Cu at (148.5, 96.9)
