File: Pavel/Tuerschild_Boarddesign.sch (KiCad schematic (older format))
At the start: 0 parts

Commit message: save commit again
Parts:
- added J101: Conn_01x02_Male, Pavel_privat:Batterieeinspeisungspads, symbol Connector:Conn_01x02_Male
Connections:
- net +BATT: now also J101.1 (Pin_1)
- net GNDPWR: now also J101.2 (Pin_2)
