File: Hardware/IO-Platine.sch (KiCad schematic (older format))
At the start: 9 parts, among them J501 S8B-PH-SM4-TB, J502 Con.2-Pol

Commit message: finished PCB, Thursday Review with Lukas
Parts:
- R502: renamed from R?; footprint Resistor_SMD:R_0805_2012Metric_Pad1.15x1.40mm_HandSolder -> Resistor_SMD:R_0805_2012Metric_Pad1.20x1.40mm_HandSolder
Changed lines of the file:
@@
 AR Path="/5F894235" Ref="#PWR?"  Part="1"
 AR Path="/5DE5A7F7/5F894235" Ref="#PWR?"  Part="1"
-AR Path="/5DE7403E/5F894235" Ref="#PWR?"  Part="1"
-F 0 "#PWR?" H 9150 2900 50  0001 C CNN
+AR Path="/5DE7403E/5F894235" Ref="#PWR0121"  Part="1"
+F 0 "#PWR0121" H 9150 2900 50  0001 C CNN
 F 1 "+3V3" H 9165 3223 50  0000 C CNN
 F 2 "" H 9150 3050 50  0001 C CNN
@@
 AR Path="/5F89423B" Ref="R?"  Part="1"
 AR Path="/5DE4BC0A/5F89423B" Ref="R?"  Part="1"
-AR Path="/5DE7403E/5F89423B" Ref="R?"  Part="1"
-F 0 "R?" V 9254 3178 50  0000 L CNN
+AR Path="/5DE7403E/5F89423B" Ref="R502"  Part="1"
+F 0 "R502" V 9254 3178 50  0000 L CNN
 F 1 "4k7" V 9345 3178 50  0000 L CNN
-F 2 "Resistor_SMD:R_0805_2012Metric_Pad1.15x1.40mm_HandSolder" H 9250 3000 50  0001 C CNN
+F 2 "Resistor_SMD:R_0805_2012Metric_Pad1.20x1.40mm_HandSolder" H 9250 3000 50  0001 C CNN
 F 3 "" H 9200 3200 50  0001 C CNN
 	1    9200 3150
