File: Hardware/E-Ink.kicad_pcb (KiCad board)
At the start: 2 copper layers, 65.2 x 56.2 mm, 64 parts, among them J501 S8B-PH-SM4-TB, J502 Con.2-Pol, Q201 2N7000, Q301 2N7000, U201 TPS63002DRCR, U202 TPS63031DSKR, U401 ESP32-WROOM-32U, U501 TXB0104PWR

Commit message: savecommit
Parts:
- R501: value 47k -> 4k7
Connections:
- S501 pad 1: (no net) -> Net-(S501-Pad1)
- S501 pad 3: (no net) -> Net-(S501-Pad3)
- S502 pad 1: (no net) -> Net-(S502-Pad1)
- S502 pad 3: (no net) -> Net-(S502-Pad3)
- U401 pad 17: (no net) -> Net-(U401-Pad17)
- U401 pad 18: (no net) -> Net-(U401-Pad18)
- U401 pad 19: (no net) -> Net-(U401-Pad19)
- U401 pad 20: (no net) -> Net-(U401-Pad20)
- U401 pad 21: (no net) -> Net-(U401-Pad21)
- U401 pad 22: (no net) -> Net-(U401-Pad22)
- U401 pad 24: (no net) -> Net-(U401-Pad24)
- U401 pad 26: (no net) -> Net-(U401-Pad26)
- U401 pad 29: (no net) -> Net-(U401-Pad29)
- U401 pad 30: (no net) -> Net-(U401-Pad30)
- U401 pad 31: (no net) -> Net-(U401-Pad31)
- U401 pad 32: (no net) -> Net-(U401-Pad32)
- U401 pad 37: (no net) -> Net-(U401-Pad37)
- U401 pad 5: (no net) -> Net-(U401-Pad5)
- U401 pad 6: (no net) -> Net-(U401-Pad6)
- U401 pad 7: (no net) -> Net-(U401-Pad7)
- U501 pad 6: (no net) -> Net-(U501-Pad6)
- U501 pad 9: (no net) -> Net-(U501-Pad9)
Routing:
- net GND: track 30.3 -> 41.9 mm, vias 2 -> 4
