File: Hardware/E-Ink.kicad_pcb (KiCad board)
At the start: 2 copper layers, 65.2 x 56.2 mm, 64 parts, among them J501 S8B-PH-SM4-TB, J502 Con.2-Pol, Q201 2N7000, Q301 2N7000, U201 TPS63002DRCR, U202 TPS63031DSKR, U401 ESP32-WROOM-32U, U501 TXB0104PWR

Commit message: finished PCB and ordered
Other:
- board text added: "3V3"
- board text added: "5V"
- board text added: "CS"
- board text added: "E-Ink-Parkplatzanzeige V10 OTH-Regensburg Labor IE VMCB WS19/20 Martin Brandl, Simon Schindler"
- board text added: "GND"
- board text added: "MISO"
- board text added: "MOSI"
- board text added: "SCK"
Changed lines of the file:
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@@
   (general
     (thickness 1.6)
-    (drawings 8)
+    (drawings 16)
     (tracks 455)
     (zones 0)
@@
     (0 F.Cu signal)
     (31 B.Cu signal)
-    (32 B.Adhes user)
-    (33 F.Adhes user)
-    (34 B.Paste user)
-    (35 F.Paste user)
+    (32 B.Adhes user hide)
+    (33 F.Adhes user hide)
+    (34 B.Paste user hide)
+    (35 F.Paste user hide)
     (36 B.SilkS user)
     (37 F.SilkS user)
     (38 B.Mask user)
     (39 F.Mask user)
-    (40 Dwgs.User user)
-    (41 Cmts.User user)
-    (42 Eco1.User user)
-    (43 Eco2.User user)
+    (40 Dwgs.User user hide)
+    (41 Cmts.User user hide)
+    (42 Eco1.User user hide)
+    (43 Eco2.User user hide)
     (44 Edge.Cuts user)
-    (45 Margin user)
-    (46 B.CrtYd user)
-    (47 F.CrtYd user)
-    (48 B.Fab user)
+    (45 Margin user hide)
+    (46 B.CrtYd user hide)
+    (47 F.CrtYd user hide)
+    (48 B.Fab user hide)
     (49 F.Fab user hide)
   )
@@
     (mod_text_size 1 1)
     (mod_text_width 0.15)
-    (pad_size 1.524 1.524)
-    (pad_drill 0.762)
+    (pad_size 2.02 2.02)
+    (pad_drill 1.02)
     (pad_to_mask_clearance 0.051)
     (solder_mask_min_width 0.4)
     (aux_axis_origin 0 0)
-    (grid_origin 9.3 8.02)
+    (grid_origin 92.3 70.22)
     (visible_elements 7FFFFFFF)
     (pcbplotparams
-      (layerselection 0x010fc_ffffffff)
-      (usegerberextensions false)
+      (layerselection 0x010f0_ffffffff)
+      (usegerberextensions true)
       (usegerberattributes false)
       (usegerberadvancedattributes false)
@@
       (outputformat 1)
       (mirror false)
-      (drillshape 1)
+      (drillshape 0)
       (scaleselection 1)
-      (outputdirectory ""))
+      (outputdirectory "Output/Drill"))
   )
   (net 0 "")
@@
     (pad 1 smd rect (at -1.95 2.875) (size 0.35 1.4) (layers F.Cu F.Paste F.Mask)
       (net 20 +3V3))
+  )
+  (gr_text CS (at 129.4 95) (layer F.SilkS)
+    (effects (font (size 1 1) (thickness 0.15)))
+  )
+  (gr_text SCK (at 125.9 95) (layer F.SilkS)
+    (effects (font (size 1 1) (thickness 0.15)))
+  )
+  (gr_text MOSI (at 122.4 95) (layer F.SilkS)
+    (effects (font (size 1 1) (thickness 0.15)))
+  )
+  (gr_text MISO (at 118.9 95) (layer F.SilkS)
+    (effects (font (size 1 1) (thickness 0.15)))
+  )
+  (gr_text 5V (at 115.4 95) (layer F.SilkS)
+    (effects (font (size 1 1) (thickness 0.15)))
+  )
+  (gr_text 3V3 (at 111.9 95) (layer F.SilkS)
+    (effects (font (size 1 1) (thickness 0.15)))
+  )
+  (gr_text GND (at 108.3 95) (layer F.SilkS)
+    (effects (font (size 1 1) (thickness 0.15)))
+  )
+  (gr_text "E-Ink-Parkplatzanzeige V10\nOTH-Regensburg\nLabor IE\nVMCB WS19/20\nMartin Brandl, Simon Schindler" (at 153.1 86.22 90) (layer B.Mask)
+    (effects (font (size 1 1) (thickness 0.15)) (justify mirror))
   )
   (gr_circle (center 161.7 47.31) (end 161.7 48.81) (layer Edge.Cuts) (width 0.05))
@@
   (segment (start 110.31 59.45) (end 107.895 59.45) (width 0.1524) (layer F.Cu) (net 25))
   (via (at 127.8 76.02) (size 0.8) (drill 0.4) (layers F.Cu B.Cu) (net 26))
-  (segment (start 129.3 97.52) (end 129.3 77.52) (width 0.1524) (layer B.Cu) (net 26))
   (segment (start 129.3 77.52) (end 127.8 76.02) (width 0.1524) (layer B.Cu) (net 26))
   (segment (start 127.8 73.82) (end 127.855 73.765) (width 0.1524) (layer F.Cu) (net 26))
@@
   (segment (start 132.119488 68.884827) (end 131.4 68.165339) (width 0.1524) (layer F.Cu) (net 26))
   (segment (start 132.119488 69.450512) (end 132.119488 68.884827) (width 0.1524) (layer F.Cu) (net 26))
+  (segment (start 129.3 97.52) (end 129.3 77.52) (width 0.1524) (layer B.Cu) (net 26))
   (segment (start 119.676628 82.121628) (end 115.651628 82.121628) (width 0.1524) (layer F.Cu) (net 27))
   (segment (start 120.3 82.745) (end 119.676628 82.121628) (width 0.1524) (layer F.Cu) (net 27))

Commit message: Save work at Arges
Connections:
- S501 pad 1: Net-(S501-Pad1) -> (no net)
- S501 pad 3: Net-(S501-Pad3) -> (no net)
- S502 pad 1: Net-(S502-Pad1) -> (no net)
- S502 pad 3: Net-(S502-Pad3) -> (no net)
- U401 pad 17: Net-(U401-Pad17) -> (no net)
- U401 pad 18: Net-(U401-Pad18) -> (no net)
- U401 pad 19: Net-(U401-Pad19) -> (no net)
- U401 pad 20: Net-(U401-Pad20) -> (no net)
- U401 pad 21: Net-(U401-Pad21) -> (no net)
- U401 pad 22: Net-(U401-Pad22) -> (no net)
- U401 pad 24: Net-(U401-Pad24) -> (no net)
- U401 pad 26: Net-(U401-Pad26) -> (no net)
- U401 pad 29: Net-(U401-Pad29) -> (no net)
- U401 pad 30: Net-(U401-Pad30) -> (no net)
- U401 pad 31: Net-(U401-Pad31) -> (no net)
- U401 pad 32: Net-(U401-Pad32) -> (no net)
- U401 pad 37: Net-(U401-Pad37) -> (no net)
- U401 pad 5: Net-(U401-Pad5) -> (no net)
- U401 pad 6: Net-(U401-Pad6) -> (no net)
- U401 pad 7: Net-(U401-Pad7) -> (no net)
- U501 pad 6: Net-(U501-Pad6) -> (no net)
- U501 pad 9: Net-(U501-Pad9) -> (no net)
Routing:
- net SCK: track 59.9 -> 55.3 mm
- net CS: track 36.1 -> 33.2 mm
Changed lines of the file:
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@@
-(kicad_pcb (version 20171130) (host pcbnew 5.1.5-52549c5~84~ubuntu18.04.1)
+(kicad_pcb (version 20171130) (host pcbnew "(5.1.4)-1")
   (general
     (thickness 1.6)
     (drawings 16)
-    (tracks 455)
+    (tracks 453)
     (zones 0)
     (modules 64)
-    (nets 63)
+    (nets 41)
   )
   (page A4)
@@
   (net 39 MOSI)
   (net 40 SCK)
-  (net 41 "Net-(S501-Pad1)")
-  (net 42 "Net-(S501-Pad3)")
-  (net 43 "Net-(S502-Pad3)")
-  (net 44 "Net-(S502-Pad1)")
-  (net 45 "Net-(U401-Pad5)")
-  (net 46 "Net-(U401-Pad6)")
-  (net 47 "Net-(U401-Pad7)")
-  (net 48 "Net-(U401-Pad17)")
-  (net 49 "Net-(U401-Pad18)")
-  (net 50 "Net-(U401-Pad19)")
-  (net 51 "Net-(U401-Pad20)")
-  (net 52 "Net-(U401-Pad21)")
-  (net 53 "Net-(U401-Pad22)")
-  (net 54 "Net-(U401-Pad24)")
-  (net 55 "Net-(U401-Pad26)")
-  (net 56 "Net-(U401-Pad29)")
-  (net 57 "Net-(U401-Pad30)")
-  (net 58 "Net-(U401-Pad31)")
-  (net 59 "Net-(U401-Pad32)")
-  (net 60 "Net-(U401-Pad37)")
-  (net 61 "Net-(U501-Pad6)")
-  (net 62 "Net-(U501-Pad9)")
   (net_class Default "This is the default net class."
     (clearance 0.1524)
@@
     (pad 38 smd rect (at 8.5 -8.255 180) (size 2 0.9) (layers F.Cu F.Paste F.Mask)
       (net 1 GND))
-    (pad 37 smd rect (at 8.5 -6.985 180) (size 2 0.9) (layers F.Cu F.Paste F.Mask)
-      (net 60 "Net-(U401-Pad37)"))
+    (pad 37 smd rect (at 8.5 -6.985 180) (size 2 0.9) (layers F.Cu F.Paste F.Mask))
     (pad 36 smd rect (at 8.5 -5.715 180) (size 2 0.9) (layers F.Cu F.Paste F.Mask)
       (net 22 "Net-(R403-Pad2)"))
@@
     (pad 33 smd rect (at 8.5 -1.905 180) (size 2 0.9) (layers F.Cu F.Paste F.Mask)
       (net 21 "Net-(R402-Pad1)"))
-    (pad 32 smd rect (at 8.5 -0.635 180) (size 2 0.9) (layers F.Cu F.Paste F.Mask)
-      (net 59 "Net-(U401-Pad32)"))
-    (pad 31 smd rect (at 8.5 0.635 180) (size 2 0.9) (layers F.Cu F.Paste F.Mask)
-      (net 58 "Net-(U401-Pad31)"))
-    (pad 30 smd rect (at 8.5 1.905 180) (size 2 0.9) (layers F.Cu F.Paste F.Mask)
-      (net 57 "Net-(U401-Pad30)"))
-    (pad 29 smd rect (at 8.5 3.175 180) (size 2 0.9) (layers F.Cu F.Paste F.Mask)
-      (net 56 "Net-(U401-Pad29)"))
+    (pad 32 smd rect (at 8.5 -0.635 180) (size 2 0.9) (layers F.Cu F.Paste F.Mask))
+    (pad 31 smd rect (at 8.5 0.635 180) (size 2 0.9) (layers F.Cu F.Paste F.Mask))
+    (pad 30 smd rect (at 8.5 1.905 180) (size 2 0.9) (layers F.Cu F.Paste F.Mask))
+    (pad 29 smd rect (at 8.5 3.175 180) (size 2 0.9) (layers F.Cu F.Paste F.Mask))
     (pad 28 smd rect (at 8.5 4.445 180) (size 2 0.9) (layers F.Cu F.Paste F.Mask)
       (net 11 EN_5V))
     (pad 27 smd rect (at 8.5 5.715 180) (size 2 0.9) (layers F.Cu F.Paste F.Mask)
       (net 16 EN_Vmess))
-    (pad 26 smd rect (at 8.5 6.985 180) (size 2 0.9) (layers F.Cu F.Paste F.Mask)
-      (net 55 "Net-(U401-Pad26)"))
+    (pad 26 smd rect (at 8.5 6.985 180) (size 2 0.9) (layers F.Cu F.Paste F.Mask))
     (pad 25 smd rect (at 8.5 8.255 180) (size 2 0.9) (layers F.Cu F.Paste F.Mask)
       (net 23 PROG_ESP))
-    (pad 24 smd rect (at 5.715 9.255 270) (size 2 0.9) (layers F.Cu F.Paste F.Mask)
-      (net 54 "Net-(U401-Pad24)"))
+    (pad 24 smd rect (at 5.715 9.255 270) (size 2 0.9) (layers F.Cu F.Paste F.Mask))
     (pad 23 smd rect (at 4.445 9.255 270) (size 2 0.9) (layers F.Cu F.Paste F.Mask)
       (net 26 CS))
-    (pad 22 smd rect (at 3.175 9.255 270) (size 2 0.9) (layers F.Cu F.Paste F.Mask)
-      (net 53 "Net-(U401-Pad22)"))
-    (pad 21 smd rect (at 1.905 9.255 270) (size 2 0.9) (layers F.Cu F.Paste F.Mask)
-      (net 52 "Net-(U401-Pad21)"))
-    (pad 20 smd rect (at 0.635 9.255 270) (size 2 0.9) (layers F.Cu F.Paste F.Mask)
-      (net 51 "Net-(U401-Pad20)"))
-    (pad 19 smd rect (at -0.635 9.255 270) (size 2 0.9) (layers F.Cu F.Paste F.Mask)
-      (net 50 "Net-(U401-Pad19)"))
-    (pad 18 smd rect (at -1.905 9.255 270) (size 2 0.9) (layers F.Cu F.Paste F.Mask)
-      (net 49 "Net-(U401-Pad18)"))
-    (pad 17 smd rect (at -3.175 9.255 270) (size 2 0.9) (layers F.Cu F.Paste F.Mask)
-      (net 48 "Net-(U401-Pad17)"))
+    (pad 22 smd rect (at 3.175 9.255 270) (size 2 0.9) (layers F.Cu F.Paste F.Mask))
+    (pad 21 smd rect (at 1.905 9.255 270) (size 2 0.9) (layers F.Cu F.Paste F.Mask))
+    (pad 20 smd rect (at 0.635 9.255 270) (size 2 0.9) (layers F.Cu F.Paste F.Mask))
+    (pad 19 smd rect (at -0.635 9.255 270) (size 2 0.9) (layers F.Cu F.Paste F.Mask))
+    (pad 18 smd rect (at -1.905 9.255 270) (size 2 0.9) (layers F.Cu F.Paste F.Mask))
+    (pad 17 smd rect (at -3.175 9.255 270) (size 2 0.9) (layers F.Cu F.Paste F.Mask))
     (pad 16 smd rect (at -4.445 9.255 270) (size 2 0.9) (layers F.Cu F.Paste F.Mask)
       (net 39 MOSI))
@@
     (pad 8 smd rect (at -8.5 0.635 180) (size 2 0.9) (layers F.Cu F.Paste F.Mask)
       (net 36 "Net-(TP406-Pad1)"))
-    (pad 7 smd rect (at -8.5 -0.635 180) (size 2 0.9) (layers F.Cu F.Paste F.Mask)
-      (net 47 "Net-(U401-Pad7)"))
-    (pad 6 smd rect (at -8.5 -1.905 180) (size 2 0.9) (layers F.Cu F.Paste F.Mask)
-      (net 46 "Net-(U401-Pad6)"))
-    (pad 5 smd rect (at -8.5 -3.175 180) (size 2 0.9) (layers F.Cu F.Paste F.Mask)
-      (net 45 "Net-(U401-Pad5)"))
+    (pad 7 smd rect (at -8.5 -0.635 180) (size 2 0.9) (layers F.Cu F.Paste F.Mask))
+    (pad 6 smd rect (at -8.5 -1.905 180) (size 2 0.9) (layers F.Cu F.Paste F.Mask))
+    (pad 5 smd rect (at -8.5 -3.175 180) (size 2 0.9) (layers F.Cu F.Paste F.Mask))
     (pad 4 smd rect (at -8.5 -4.445 180) (size 2 0.9) (layers F.Cu F.Paste F.Mask)
       (net 2 GPIO_Vmess))
@@
       (effects (font (size 1 1) (thickness 0.15)))
     )
-    (pad 1 smd rect (at -4.55 -2.25 270) (size 1.4 2.1) (layers F.Cu F.Paste F.Mask)
-      (net 41 "Net-(S501-Pad1)"))
-    (pad 3 smd rect (at -4.55 2.25 270) (size 1.4 2.1) (layers F.Cu F.Paste F.Mask)
-      (net 42 "Net-(S501-Pad3)"))
+    (pad 1 smd rect (at -4.55 -2.25 270) (size 1.4 2.1) (layers F.Cu F.Paste F.Mask))
+    (pad 3 smd rect (at -4.55 2.25 270) (size 1.4 2.1) (layers F.Cu F.Paste F.Mask))
     (pad 4 smd rect (at 4.55 2.25 270) (size 1.4 2.1) (layers F.Cu F.Paste F.Mask)
       (net 1 GND))
@@
       (effects (font (size 1 1) (thickness 0.15)))
     )
-    (pad 1 smd rect (at -4.55 -2.25 270) (size 1.4 2.1) (layers F.Cu F.Paste F.Mask)
-      (net 44 "Net-(S502-Pad1)"))
-    (pad 3 smd rect (at -4.55 2.25 270) (size 1.4 2.1) (layers F.Cu F.Paste F.Mask)
-      (net 43 "Net-(S502-Pad3)"))
+    (pad 1 smd rect (at -4.55 -2.25 270) (size 1.4 2.1) (layers F.Cu F.Paste F.Mask))
+    (pad 3 smd rect (at -4.55 2.25 270) (size 1.4 2.1) (layers F.Cu F.Paste F.Mask))
     (pad 4 smd rect (at 4.55 2.25 270) (size 1.4 2.1) (layers F.Cu F.Paste F.Mask)
       (net 1 GND))
@@
     (pad 8 smd rect (at 1.95 -2.875) (size 0.35 1.4) (layers F.Cu F.Paste F.Mask)
       (net 11 EN_5V))
-    (pad 9 smd rect (at 1.3 -2.875) (size 0.35 1.4) (layers F.Cu F.Paste F.Mask)
-      (net 62 "Net-(U501-Pad9)"))
+    (pad 9 smd rect (at 1.3 -2.875) (size 0.35 1.4) (layers F.Cu F.Paste F.Mask))
     (pad 10 smd rect (at 0.65 -2.875) (size 0.35 1.4) (layers F.Cu F.Paste F.Mask)
       (net 32 "Net-(J501-Pad3)"))
@@
     (pad 7 smd rect (at 1.95 2.875) (size 0.35 1.4) (layers F.Cu F.Paste F.Mask)
       (net 1 GND))
-    (pad 6 smd rect (at 1.3 2.875) (size 0.35 1.4) (layers F.Cu F.Paste F.Mask)
-      (net 61 "Net-(U501-Pad6)"))
+    (pad 6 smd rect (at 1.3 2.875) (size 0.35 1.4) (layers F.Cu F.Paste F.Mask))
     (pad 5 smd rect (at 0.65 2.875) (size 0.35 1.4) (layers F.Cu F.Paste F.Mask)
       (net 38 MISO))
@@
   (segment (start 130.8 70.77) (end 132.119488 69.450512) (width 0.1524) (layer B.Cu) (net 26))
   (segment (start 131.4 65.2474) (end 131.4 64.395) (width 0.1524) (layer F.Cu) (net 26))
-  (segment (start 131.4 68.165339) (end 131.4 65.2474) (width 0.1524) (layer F.Cu) (net 26))
   (segment (start 132.119488 68.884827) (end 131.4 68.165339) (width 0.1524) (layer F.Cu) (net 26))
   (segment (start 132.119488 69.450512) (end 132.119488 68.884827) (width 0.1524) (layer F.Cu) (net 26))
@@
   (via (at 133.3 71.52) (size 0.8) (drill 0.4) (layers F.Cu B.Cu) (net 40))
   (segment (start 142.73033 71.52) (end 133.3 71.52) (width 0.1524) (layer B.Cu) (net 40))
-  (segment (start 130.75 68.97) (end 130.75 64.395) (width 0.1524) (layer F.Cu) (net 40))
   (segment (start 133.3 71.52) (end 130.75 68.97) (width 0.1524) (layer F.Cu) (net 40))
   (segment (start 128.199999 95.120001) (end 128.199999 79.669999) (width 0.1524) (layer B.Cu) (net 40))

Commit message: finished PCB, Thursday Review with Lukas
Parts:
- removed C501, C502: 100n, Capacitor_SMD:C_0805_2012Metric_Pad1.15x1.40mm_HandSolder
- removed Q201, Q301: 2N7000, Digikey:TO-92-3
- removed R201: 4k7, Resistor_SMD:R_0805_2012Metric_Pad1.15x1.40mm_HandSolder
- removed R202: 47k, Resistor_SMD:R_0805_2012Metric_Pad1.15x1.40mm_HandSolder
- removed R303, R304, R402, R403: 0, Resistor_SMD:R_0805_2012Metric_Pad1.15x1.40mm_HandSolder
- removed U501: TXB0104PWR, Digikey:TSSOP-14_W4.4mm
- added R502: 4k7, Resistor_SMD:R_0805_2012Metric_Pad1.20x1.40mm_HandSolder, F.Cu at (151.2, 72.9)
- R301: value 4k7 -> 10M; footprint Resistor_SMD:R_0805_2012Metric_Pad1.15x1.40mm_HandSolder -> Resistor_SMD:R_0805_2012Metric_Pad1.20x1.40mm_HandSolder
- R302: value 47k -> 10M; footprint Resistor_SMD:R_0805_2012Metric_Pad1.15x1.40mm_HandSolder -> Resistor_SMD:R_0805_2012Metric_Pad1.20x1.40mm_HandSolder
- U401: value ESP32-WROOM-32U -> ESP-32-WROOVER-IE; footprint RF_Module:ESP32-WROOM-32U -> E-Ink:ESP32-WROVER
- moved R501 29.5 mm to (147.5, 72.9)
- moved C504 24.8 mm to (145.1, 72.9)
- moved U401 5.79 mm to (127.9, 86.7)
- moved R301 5.21 mm to (110.7, 47.0), turned to 90 degrees
- moved R302 4.61 mm to (115.2, 47.0), turned to 90 degrees
- moved C301 0.21 mm to (113.0, 47.0)
- moved C302 0.05 mm to (117.3, 47.0)
Connections:
- C301 pad 1: Net-(C301-Pad1) -> +BATT
- J501 pad 3: Net-(J501-Pad3) -> MISO
- J501 pad 4: Net-(J501-Pad4) -> MOSI
- J501 pad 5: Net-(J501-Pad5) -> SCK
- J501 pad 6: Net-(J501-Pad6) -> CS
- R203 pad 1: Net-(Q201-Pad1) -> EN_5V
- R301 pad 1: Net-(Q301-Pad2) -> GPIO_Vmess
- R301 pad 2: EN_Vmess -> +BATT
- R302 pad 1: Net-(C301-Pad1) -> GPIO_Vmess
- R302 pad 2: Net-(Q301-Pad2) -> GND
- S501 pad 1: (no net) -> Net-(S501-Pad1)
- S501 pad 3: (no net) -> Net-(S501-Pad3)
- S502 pad 1: (no net) -> Net-(S502-Pad1)
- S502 pad 3: (no net) -> Net-(S502-Pad3)
- U201 pad 6: Net-(Q201-Pad1) -> EN_5V
- U401 pad 10: Net-(TP403-Pad1) -> Net-(TP404-Pad1)
- U401 pad 11: Net-(TP404-Pad1) -> Net-(TP403-Pad1)
- U401 pad 12: Net-(TP405-Pad1) -> Net-(U401-Pad12)
- U401 pad 15: GND -> Net-(U401-Pad15)
- U401 pad 17: (no net) -> Net-(U401-Pad17)
- U401 pad 18: (no net) -> Net-(U401-Pad18)
- U401 pad 19: (no net) -> Net-(U401-Pad19)
- U401 pad 20: (no net) -> Net-(U401-Pad20)
- U401 pad 21: (no net) -> Net-(U401-Pad21)
- U401 pad 22: (no net) -> Net-(U401-Pad22)
- U401 pad 24: (no net) -> Net-(U401-Pad24)
- U401 pad 26: (no net) -> Net-(U401-Pad26)
- U401 pad 27: EN_Vmess -> Net-(U401-Pad27)
- U401 pad 28: EN_5V -> Net-(U401-Pad28)
- U401 pad 29: (no net) -> EN_5V
- U401 pad 30: (no net) -> Net-(U401-Pad30)
- U401 pad 31: (no net) -> Net-(U401-Pad31)
- U401 pad 32: (no net) -> Net-(U401-Pad32)
- U401 pad 33: Net-(R402-Pad1) -> BSY_DIS
- U401 pad 36: Net-(R403-Pad2) -> RST_DIS
- U401 pad 37: (no net) -> Net-(U401-Pad37)
- U401 pad 39: (no net) -> GND
- U401 pad 5: (no net) -> GND
- U401 pad 6: (no net) -> Net-(U401-Pad6)
- U401 pad 7: (no net) -> Net-(TP407-Pad1)
- U401 pad 9: Net-(TP407-Pad1) -> Net-(TP405-Pad1)
Routing:
- net EN_Vmess: track 38.3 -> 0.00 mm, vias 4 -> 0
- net +3V3: track 43.2 -> 80.9 mm, vias 4 -> 2
- net RST_ESP: track 23.9 -> 52.9 mm, vias 0 -> 2
- net CS: track 33.2 -> 61.2 mm, vias 3 -> 5
- net Net-(Q201-Pad1): track 24.5 -> 0.00 mm, vias 2 -> 0
- net +BATT: track 107.0 -> 122.0 mm
- net Net-(R204-Pad2): track 27.4 -> 13.6 mm, vias 0 -> 2
- net MOSI: track 46.9 -> 59.3 mm, vias 1 -> 5
- net Net-(C301-Pad1): track 12.0 -> 0.00 mm
- net BSY_DIS: track 44.3 -> 32.6 mm, vias 2 -> 4
- net TXD0: track 25.5 -> 14.4 mm
- net RST_DIS: track 49.0 -> 38.0 mm, vias 4 -> 6
- net Net-(Q201-Pad2): track 9.26 -> 0.00 mm, vias 1 -> 0
- net Net-(TP406-Pad1): track 28.9 -> 37.5 mm, vias 0 -> 2
- net Net-(Q301-Pad2): track 8.21 -> 0.00 mm
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Other:
- rule via_min_size: 0.4 -> 0.45

Commit message: added all changes just to make sure
Routing:
- net +BATT: track 122.0 -> 128.3 mm
- net Net-(TP405-Pad1): track 44.1 -> 49.4 mm, vias 2 -> 3
- net +3V3: track 80.9 -> 82.2 mm
- net +5V: track 92.7 -> 93.3 mm
Other:
- net class Default: clearance 0.1524 -> 0.254
- net class Power: clearance 0.1524 -> 0.254
- rule trace_clearance: 0.1524 -> 0.254
