File: Hardware/ESP 32 Modul.sch (KiCad schematic (older format))
At the start: 6 parts

Commit message: save commit
Parts:
- removed R?: 10k, Resistor_SMD:R_0805_2012Metric_Pad1.15x1.40mm_HandSolder, symbol E-Ink:10k
- added R?: 47k, Resistor_SMD:R_0805_2012Metric_Pad1.15x1.40mm_HandSolder, symbol E-Ink:47k
Connections:
- net +3V3: now also R?.1
- net Reset_ESP: now also R?.2
- net PROG_ESP: now reaches U?.25 (IO0)
- net RXD0: now reaches U?.34 (RXD0/IO3)
- net TXD0: now reaches U?.35 (TXD0/IO1)
Other:
- note added: "Schwacher PU zum Energiesparen. \nEventuell stärkeren PU einsetzen."
Changed lines of the file:
@@
 	1    0    0    -1
-$EndComp
-$Comp
-L E-Ink:10k R?
-U 1 1 5DE6A494
-P 2600 1850
-AR Path="/5DE6A494" Ref="R?"  Part="1"
-AR Path="/5DE5A7F7/5DE6A494" Ref="R?"  Part="1"
-F 0 "R?" V 2654 1878 50  0000 L CNN
-F 1 "10k" V 2745 1878 50  0000 L CNN
-F 2 "Resistor_SMD:R_0805_2012Metric_Pad1.15x1.40mm_HandSolder" H 2650 1700 50  0001 C CNN
-F 3 "" H 2600 1900 50  0001 C CNN
-	1    2600 1850
-	0    1    1    0
 $EndComp
 Wire Wire Line
@@
 Wire Wire Line
 	1500 1950 1400 1950
+Text HLabel 4150 2300 2    50   Input ~ 10
+PROG_ESP
+Text HLabel 4150 2400 2    50   Output ~ 10
+TXD0
+Text HLabel 4150 2600 2    50   Input ~ 10
+RXD0
+$Comp
+L E-Ink:47k R?
+U 1 1 5DE23BF7
+P 2600 1850
+AR Path="/5DE23BF7" Ref="R?"  Part="1"
+AR Path="/5DE4BC0A/5DE23BF7" Ref="R?"  Part="1"
+AR Path="/5DE5A7F7/5DE23BF7" Ref="R?"  Part="1"
+F 0 "R?" V 2654 1878 50  0000 L CNN
+F 1 "47k" V 2745 1878 50  0000 L CNN
+F 2 "Resistor_SMD:R_0805_2012Metric_Pad1.15x1.40mm_HandSolder" H 2650 1700 50  0001 C CNN
+F 3 "" H 2600 1900 50  0001 C CNN
+	1    2600 1850
+	0    1    1    0
+$EndComp
+Text Notes 1950 2000 0    20   ~ 4
+Schwacher PU zum Energiesparen. \nEventuell stärkeren PU einsetzen.
 $EndSCHEMATC

Commit message: save commit from work at night
Parts:
- added C11: 10µ, Capacitor_SMD:C_0805_2012Metric_Pad1.15x1.40mm_HandSolder, symbol E-Ink:10µ
- added TP1, TP10, TP11, TP12, TP13, TP14, TP2, TP3, TP4, TP5, TP6, TP7, TP8, TP9: TestPoint, symbol E-Ink:TestPoint
- gave numbers to parts that had none: 6
Connections:
- net +3V3: now also TP1.1
- net CS: now also TP11.1
- net GND: now also C11.2, TP2.1
- net MISO: now also TP8.1
- net MOSI: now also TP9.1
- net PROG_ESP: now also TP14.1
- net RXD0: now also TP13.1
- net Reset_ESP: now also C11.1
- net SCK: now also TP10.1
- net TXD0: now also TP12.1
- net at U3.10 (IO25): now also TP3.1
- net at U3.11 (IO26): now also TP4.1
- net at U3.12 (IO27): now also TP5.1
- net at U3.8 (IO32): now also TP6.1
- net at U3.9 (IO33): now also TP7.1
Other:
- note added: "Enable the 5V Powersupply \nfor the E-Ink Display\n"
- note added: "Enable the battery-voltage \nat the measurement circuit\n"
- note added: "SPI-Interface for \nCommunication with Display\n"
- note added: "Schwacher PU zum Energiesparen. \nEventuell stärkeren PU einsetzen. \nAußerdem ist EN intern mit PU versehen.\n-> Vllt auch einfach weglassen."
- note added: "UART-Programming Interface\n"
- note removed: "Schwacher PU zum Energiesparen. \nEventuell stärkeren PU einsetzen."
- moved on the sheet: C12

Commit message: Save work from OTH
Parts:
- added R? (x2): 0, Resistor_SMD:R_0805_2012Metric_Pad1.15x1.40mm_HandSolder, symbol E-Ink:0
Connections:
- net at U3.33 (IO21): now also R?.1
- net at U3.36 (IO22): now also R?.2
- new net BSY_DIS: R?.2
- new net RST_DIS: R?.1
Other:
- note added: "PINS zur späteren evtl. Benutzung"
Changed lines of the file:
@@
 EESchema Schematic File Version 4
-EELAYER 30 0
+LIBS:E-Ink-cache
+EELAYER 29 0
 EELAYER END
 $Descr A4 11693 8268
@@
 	0    1    1    0
 $EndComp
+Text Notes 4480 3950 3    20   ~ 4
+PINS zur späteren evtl. Benutzung
+Text HLabel 5100 3850 2    50   Output ~ 10
+RST_DIS
+Wire Wire Line
+	5100 3850 5000 3850
+Text HLabel 5100 3650 2    50   Input ~ 10
+BSY_DIS
+Wire Wire Line
+	5000 3650 5100 3650
+$Comp
+L E-Ink:0 R?
+U 1 1 5DE5CA58
+P 4700 3600
+F 0 "R?" H 4800 3765 50  0000 C CNN
+F 1 "0" H 4800 3674 50  0000 C CNN
+F 2 "Resistor_SMD:R_0805_2012Metric_Pad1.15x1.40mm_HandSolder" H 4750 3450 50  0001 C CNN
+F 3 "" H 4700 3650 50  0001 C CNN
+	1    4700 3600
+	1    0    0    -1
+$EndComp
+Wire Wire Line
+	4350 3650 4350 3700
+Wire Wire Line
+	4350 3700 4150 3700
+$Comp
+L E-Ink:0 R?
+U 1 1 5DE609BB
+P 4900 3900
+F 0 "R?" H 5000 4065 50  0000 C CNN
+F 1 "0" H 5000 3974 50  0000 C CNN
+F 2 "Resistor_SMD:R_0805_2012Metric_Pad1.15x1.40mm_HandSolder" H 4950 3750 50  0001 C CNN
+F 3 "" H 4900 3950 50  0001 C CNN
+	1    4900 3900
+	-1   0    0    1
+$EndComp
+Wire Wire Line
+	4350 3800 4150 3800
+Wire Wire Line
+	4350 3800 4350 3850
+Wire Wire Line
+	4600 3650 4350 3650
+Wire Wire Line
+	4350 3850 4600 3850
 $EndSCHEMATC

Commit message: Martin ist unförmig
Parts:
- TP401: renamed from TP1; footprint (none) -> digikey-footprints:Test_Point_D1.02mm; Digi-Key_PN (none) -> 36-5001-ND
- TP402: renamed from TP2; footprint (none) -> digikey-footprints:Test_Point_D1.02mm; Digi-Key_PN (none) -> 36-5001-ND
- TP403: renamed from TP3; footprint (none) -> digikey-footprints:Test_Point_D1.02mm; Digi-Key_PN (none) -> 36-5001-ND
- TP404: renamed from TP4; footprint (none) -> digikey-footprints:Test_Point_D1.02mm; Digi-Key_PN (none) -> 36-5001-ND
- TP405: renamed from TP5; footprint (none) -> digikey-footprints:Test_Point_D1.02mm; Digi-Key_PN (none) -> 36-5001-ND
- TP406: renamed from TP6; footprint (none) -> digikey-footprints:Test_Point_D1.02mm; Digi-Key_PN (none) -> 36-5001-ND
- TP407: renamed from TP7; footprint (none) -> digikey-footprints:Test_Point_D1.02mm; Digi-Key_PN (none) -> 36-5001-ND
- TP408: renamed from TP8; footprint (none) -> digikey-footprints:Test_Point_D1.02mm; Digi-Key_PN (none) -> 36-5001-ND
- TP409: renamed from TP9; footprint (none) -> digikey-footprints:Test_Point_D1.02mm; Digi-Key_PN (none) -> 36-5001-ND
- TP410: renamed from TP10; footprint (none) -> digikey-footprints:Test_Point_D1.02mm; Digi-Key_PN (none) -> 36-5001-ND
- TP411: renamed from TP11; footprint (none) -> digikey-footprints:Test_Point_D1.02mm; Digi-Key_PN (none) -> 36-5001-ND
- TP412: renamed from TP12; footprint (none) -> digikey-footprints:Test_Point_D1.02mm; Digi-Key_PN (none) -> 36-5001-ND
- TP413: renamed from TP13; footprint (none) -> digikey-footprints:Test_Point_D1.02mm; Digi-Key_PN (none) -> 36-5001-ND
- TP414: renamed from TP14; footprint (none) -> digikey-footprints:Test_Point_D1.02mm; Digi-Key_PN (none) -> 36-5001-ND
- U401: renamed from U3; Digi-Key_PN (none) -> 1904-1028-1-ND; Distributor Digikey -> (none); Distributor Part Number 1904-1028-1-ND -> (none)
- gave numbers to parts that had none: 2
- renumbered C11 to C401, C12 to C402, C13 to C403, C14 to C404, C15 to C405, R7 to R401
Other:
- moved on the sheet: C401, C402, C403, C404, C405, R401, R402, R403, TP401, TP402, TP403, TP404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

Commit message: Ich hoffe wir koennen jetzt den Master mergen!
Other:
- note added: "Diode für schnellere Entladung \ndes Kondensators"
Changed lines of the file:
@@
 	1    0    0    -1
 $EndComp
+Text Notes 1450 3350 0    20   ~ 4
+Diode für schnellere Entladung \ndes Kondensators
 $EndSCHEMATC

Commit message: Zwischenspeicher Arbeit OTH
Parts:
- removed R401: 47k, Resistor_SMD:R_0805_2012Metric_Pad1.15x1.40mm_HandSolder, symbol E-Ink:47k
- added R401: 4k7, Resistor_SMD:R_0805_2012Metric_Pad1.15x1.40mm_HandSolder, symbol E-Ink:4k7
Connections:
- net +3V3: now also R401.1
- net Reset_ESP: now also R401.2
Other:
- note removed: "Diode für schnellere Entladung \ndes Kondensators"
- note removed: "Schwacher PU zum Energiesparen. \nEventuell stärkeren PU einsetzen. \nAußerdem ist EN intern mit PU versehen.\n-> Vllt auch einfach weglassen."
Changed lines of the file:
@@
 EESchema Schematic File Version 4
-EELAYER 30 0
+LIBS:E-Ink-cache
+EELAYER 29 0
 EELAYER END
 $Descr A4 11693 8268
@@
 Text HLabel 8900 2800 2    50   Output ~ 10
 TXD0
-Text Notes 1850 2950 0    20   ~ 4
-Schwacher PU zum Energiesparen. \nEventuell stärkeren PU einsetzen. \nAußerdem ist EN intern mit PU versehen.\n-> Vllt auch einfach weglassen.
 Wire Wire Line
 	2550 3700 2800 3700
@@
 Wire Wire Line
 	1950 3100 2150 3100
-Connection ~ 2550 3100
 Connection ~ 2150 3100
 Wire Wire Line
@@
 $EndComp
 $Comp
-L E-Ink:47k R?
-U 1 1 5DE23BF7
-P 2600 2800
-AR Path="/5DE23BF7" Ref="R?"  Part="1"
-AR Path="/5DE4BC0A/5DE23BF7" Ref="R?"  Part="1"
-AR Path="/5DE5A7F7/5DE23BF7" Ref="R401"  Part="1"
-F 0 "R401" V 2654 2828 50  0000 L CNN
-F 1 "47k" V 2745 2828 50  0000 L CNN
-F 2 "Resistor_SMD:R_0805_2012Metric_Pad1.15x1.40mm_HandSolder" H 2650 2650 50  0001 C CNN
-F 3 "" H 2600 2850 50  0001 C CNN
-	1    2600 2800
-	0    1    1    0
-$EndComp
-$Comp
 L power:GND #PWR?
 U 1 1 5DE2844D
@@
 	1    0    0    -1
 $EndComp
-Text Notes 1450 3350 0    20   ~ 4
-Diode für schnellere Entladung \ndes Kondensators
+$Comp
+L E-Ink:4k7 R401
+U 1 1 5DF2736C
+P 2600 2800
+F 0 "R401" V 2654 2828 50  0000 L CNN
+F 1 "4k7" V 2745 2828 50  0000 L CNN
+F 2 "Resistor_SMD:R_0805_2012Metric_Pad1.15x1.40mm_HandSolder" H 2650 2650 50  0001 C CNN
+F 3 "" H 2600 2850 50  0001 C CNN
+	1    2600 2800
+	0    1    1    0
+$EndComp
+Connection ~ 2550 3100
 $EndSCHEMATC

Commit message: save work at arges, finished layout and routing
Parts:
- TP401, TP402, TP403, TP404, TP405, TP406, TP407, TP408, TP409, TP410, TP411, TP412, TP413, TP414: footprint digikey-footprints:Test_Point_D1.02mm -> Digikey:Test_Point_D1.02mm
Connections:
- no-connect marks 6 -> 15
Changed lines of the file:
@@
 EESchema Schematic File Version 4
 LIBS:E-Ink-cache
-EELAYER 29 0
+EELAYER 30 0
 EELAYER END
 $Descr A4 11693 8268
@@
 F 0 "TP403" V 4208 5068 50  0000 L BNN
 F 1 "TestPoint" V 4208 4977 50  0000 R TNN
-F 2 "digikey-footprints:Test_Point_D1.02mm" H 4350 4950 50  0001 C CNN
+F 2 "Digikey:Test_Point_D1.02mm" H 4350 4950 50  0001 C CNN
 F 3 "http://www.keyelco.com/product-pdf.cfm?p=1310" H 4350 4950 50  0001 C CNN
 F 4 "36-5001-ND" H 0   0   50  0001 C CNN "Digi-Key_PN"
@@
 F 0 "TP404" V 4208 5168 50  0000 L BNN
 F 1 "TestPoint" V 4208 5077 50  0000 R TNN
-F 2 "digikey-footprints:Test_Point_D1.02mm" H 4350 5050 50  0001 C CNN
+F 2 "Digikey:Test_Point_D1.02mm" H 4350 5050 50  0001 C CNN
 F 3 "http://www.keyelco.com/product-pdf.cfm?p=1310" H 4350 5050 50  0001 C CNN
 F 4 "36-5001-ND" H 0   0   50  0001 C CNN "Digi-Key_PN"
@@
 F 0 "TP405" V 4208 5268 50  0000 L BNN
 F 1 "TestPoint" V 4208 5177 50  0000 R TNN
-F 2 "digikey-footprints:Test_Point_D1.02mm" H 4350 5150 50  0001 C CNN
+F 2 "Digikey:Test_Point_D1.02mm" H 4350 5150 50  0001 C CNN
 F 3 "http://www.keyelco.com/product-pdf.cfm?p=1310" H 4350 5150 50  0001 C CNN
 F 4 "36-5001-ND" H 0   0   50  0001 C CNN "Digi-Key_PN"
@@
 F 0 "TP406" V 4208 5368 50  0000 L BNN
 F 1 "TestPoint" V 4208 5277 50  0000 R TNN
-F 2 "digikey-footprints:Test_Point_D1.02mm" H 4350 5250 50  0001 C CNN
+F 2 "Digikey:Test_Point_D1.02mm" H 4350 5250 50  0001 C CNN
 F 3 "http://www.keyelco.com/product-pdf.cfm?p=1310" H 4350 5250 50  0001 C CNN
 F 4 "36-5001-ND" H 0   0   50  0001 C CNN "Digi-Key_PN"
@@
 F 0 "TP407" V 4208 5468 50  0000 L BNN
 F 1 "TestPoint" V 4208 5377 50  0000 R TNN
-F 2 "digikey-footprints:Test_Point_D1.02mm" H 4350 5350 50  0001 C CNN
+F 2 "Digikey:Test_Point_D1.02mm" H 4350 5350 50  0001 C CNN
 F 3 "http://www.keyelco.com/product-pdf.cfm?p=1310" H 4350 5350 50  0001 C CNN
 F 4 "36-5001-ND" H 0   0   50  0001 C CNN "Digi-Key_PN"
@@
 F 0 "TP402" H 1658 1718 50  0000 L CNN
 F 1 "TestPoint" H 1658 1627 50  0000 L CNN
-F 2 "digikey-footprints:Test_Point_D1.02mm" H 1800 1600 50  0001 C CNN
+F 2 "Digikey:Test_Point_D1.02mm" H 1800 1600 50  0001 C CNN
 F 3 "http://www.keyelco.com/product-pdf.cfm?p=1310" H 1800 1600 50  0001 C CNN
 F 4 "36-5001-ND" H 0   0   50  0001 C CNN "Digi-Key_PN"
@@
 F 0 "TP401" H 1658 1618 50  0000 L CNN
 F 1 "TestPoint" H 1658 1527 50  0000 L CNN
-F 2 "digikey-footprints:Test_Point_D1.02mm" H 1800 1500 50  0001 C CNN
+F 2 "Digikey:Test_Point_D1.02mm" H 1800 1500 50  0001 C CNN
 F 3 "http://www.keyelco.com/product-pdf.cfm?p=1310" H 1800 1500 50  0001 C CNN
 F 4 "36-5001-ND" H 0   0   50  0001 C CNN "Digi-Key_PN"
@@
 F 0 "TP411" H 7208 3168 50  0000 L CNN
 F 1 "TestPoint" H 7208 3077 50  0000 L CNN
-F 2 "digikey-footprints:Test_Point_D1.02mm" H 7350 3050 50  0001 C CNN
+F 2 "Digikey:Test_Point_D1.02mm" H 7350 3050 50  0001 C CNN
 F 3 "http://www.keyelco.com/product-pdf.cfm?p=1310" H 7350 3050 50  0001 C CNN
 F 4 "36-5001-ND" H 0   0   50  0001 C CNN "Digi-Key_PN"
@@
 F 0 "TP409" H 6408 3168 50  0000 L CNN
 F 1 "TestPoint" H 6408 3077 50  0000 L CNN
-F 2 "digikey-footprints:Test_Point_D1.02mm" H 6550 3050 50  0001 C CNN
+F 2 "Digikey:Test_Point_D1.02mm" H 6550 3050 50  0001 C CNN
 F 3 "http://www.keyelco.com/product-pdf.cfm?p=1310" H 6550 3050 50  0001 C CNN
 F 4 "36-5001-ND" H 0   0   50  0001 C CNN "Digi-Key_PN"
@@
 F 0 "TP410" H 7208 2868 50  0000 L CNN
 F 1 "TestPoint" H 7208 2777 50  0000 L CNN
-F 2 "digikey-footprints:Test_Point_D1.02mm" H 7350 2750 50  0001 C CNN
+F 2 "Digikey:Test_Point_D1.02mm" H 7350 2750 50  0001 C CNN
 F 3 "http://www.keyelco.com/product-pdf.cfm?p=1310" H 7350 2750 50  0001 C CNN
 F 4 "36-5001-ND" H 0   0   50  0001 C CNN "Digi-Key_PN"
@@
 F 0 "TP408" H 6408 2868 50  0000 L CNN
 F 1 "TestPoint" H 6408 2777 50  0000 L CNN
-F 2 "digikey-footprints:Test_Point_D1.02mm" H 6550 2750 50  0001 C CNN
+F 2 "Digikey:Test_Point_D1.02mm" H 6550 2750 50  0001 C CNN
 F 3 "http://www.keyelco.com/product-pdf.cfm?p=1310" H 6550 2750 50  0001 C CNN
 F 4 "36-5001-ND" H 0   0   50  0001 C CNN "Digi-Key_PN"
@@
 F 0 "TP414" H 9908 2868 50  0000 L CNN
 F 1 "TestPoint" H 9908 2777 50  0000 L CNN
-F 2 "digikey-footprints:Test_Point_D1.02mm" H 10050 2750 50  0001 C CNN
+F 2 "Digikey:Test_Point_D1.02mm" H 10050 2750 50  0001 C CNN
 F 3 "http://www.keyelco.com/product-pdf.cfm?p=1310" H 10050 2750 50  0001 C CNN
 F 4 "36-5001-ND" H 0   0   50  0001 C CNN "Digi-Key_PN"
@@
 F 0 "TP413" H 8908 3168 50  0000 L CNN
 F 1 "TestPoint" H 8908 3077 50  0000 L CNN
-F 2 "digikey-footprints:Test_Point_D1.02mm" H 9050 3050 50  0001 C CNN
+F 2 "Digikey:Test_Point_D1.02mm" H 9050 3050 50  0001 C CNN
 F 3 "http://www.keyelco.com/product-pdf.cfm?p=1310" H 9050 3050 50  0001 C CNN
 F 4 "36-5001-ND" H 0   0   50  0001 C CNN "Digi-Key_PN"
@@
 F 0 "TP412" H 8908 2868 50  0000 L CNN
 F 1 "TestPoint" H 8908 2777 50  0000 L CNN
-F 2 "digikey-footprints:Test_Point_D1.02mm" H 9050 2750 50  0001 C CNN
+F 2 "Digikey:Test_Point_D1.02mm" H 9050 2750 50  0001 C CNN
 F 3 "http://www.keyelco.com/product-pdf.cfm?p=1310" H 9050 2750 50  0001 C CNN
 F 4 "36-5001-ND" H 0   0   50  0001 C CNN "Digi-Key_PN"
@@
 $EndComp
 Connection ~ 2550 3100
+NoConn ~ 4150 4450
+NoConn ~ 4150 4550
+NoConn ~ 4150 4850
+NoConn ~ 4150 3450
+NoConn ~ 4150 3650
+NoConn ~ 4150 3750
+NoConn ~ 2950 3550
+NoConn ~ 4150 5550
+NoConn ~ 4150 5450
 $EndSCHEMATC
